Commit message: working on keyboard controller

File: urdf/accessories.urdf.xacro (robot description, xacro)
@@ -26,10 +26,10 @@
   </xacro:if> -->
   <!-- If enabled, generate VLP16 -->
-  <xacro:include filename="accessories/VLP-16.urdf.xacro" />
+  <!-- <xacro:include filename="accessories/VLP-16.urdf.xacro" />
   <xacro:if value="$(optenv VLP16 0)">
     <VLP16 prefix="$(optenv VLP16_MOUNT front)"
                        topic="$(optenv VLP16_TOPIC front/scan)"/>
    <link name="dummy_link"></link>
-    <joint name="$VLP16_joint" type="fixed">
+    <joint name="VLP16_joint" type="fixed">
       <origin xyz="0 0 0"
               rpy="0 0 0" />
@@ -37,5 +37,5 @@
       <child link="dummy_link" />
     </joint>
-  </xacro:if>
+  </xacro:if> -->
   <!-- If enabled, generate the upgraded Navsat payload (a Novatel Smart6). -->
   <!-- <xacro:include filename="accessories/novatel_smart6.urdf.xacro" />

File: urdf/jackal.urdf.xacro (robot description, xacro)
@@ -172,4 +172,7 @@
   <!-- Optional custom includes. -->
   <!-- <xacro:include filename="$(optenv JACKAL_URDF_EXTRAS empty.urdf)" /> -->
-  <xacro:include filename="accessories/VLP-16.urdf.xacro" />
+  <!-- <xacro:include filename="$(find velodyne_description)/urdf/VLP-16.urdf.xacro"/>
+  <VLP-16 parent="rear_mount" name="velodyne" topic="/velodyne_points">
+    <origin xyz="0 0 0.4" rpy="0 0 0" />
+  </VLP-16> -->
 </robot>
