Commit message: LIDAR working in gazebo/rviz, need to clean up unecessary files

File: urdf/jackal.urdf.xacro (robot description, xacro)
@@ -164,4 +164,20 @@
     <origin xyz="${mount_spacing} 0 0" />
   </joint>
+  <camera_mount prefix="$(optenv JACKAL_FLEA3_MOUNT front)"
+                tilt="$(optenv JACKAL_FLEA3_TILT 0.5236)"/>
+  <joint name="$(optenv JACKAL_FLEA3_MOUNT front)_camera_mount_joint" type="fixed">
+    <origin xyz="$(optenv JACKAL_FLEA3_OFFSET 0 0 0)"
+            rpy="$(optenv JACKAL_FLEA3_RPY 0 0 0)" />
+    <parent link="$(optenv JACKAL_FLEA3_MOUNT front)_mount" />
+    <child link="$(optenv JACKAL_FLEA3_MOUNT front)_camera_mount" />
+  </joint>
+  <pointgrey_flea3 frame="$(optenv JACKAL_FLEA3_MOUNT front)_camera" name="$(optenv JACKAL_FLEA3_NAME front)"
+    camera_x="0.0754" camera_y="0.029" camera_z="0.035"
+    camera_mass="0.085" hfov="1.0471975512" fps="60" width="640" height="512"/>
+  <joint name="$(optenv JACKAL_FLEA3_MOUNT front)_camera_bracket_joint" type="fixed">
+    <origin xyz="0.020 0 0.0245" rpy="0 0 0" />
+    <parent link="$(optenv JACKAL_FLEA3_MOUNT front)_camera_beam" />
+    <child link="$(optenv JACKAL_FLEA3_MOUNT front)_camera" />
+  </joint>
   <!-- Bring in simulation data for Gazebo. -->
   <xacro:include filename="jackal.gazebo" />
@@ -169,10 +185,18 @@
        of these into the final description is controlled by optenv variables, which
        default each one to off.-->
-  <xacro:include filename="accessories.urdf.xacro" />
+  <!-- <xacro:include filename="accessories.urdf.xacro" /> -->
   <!-- Optional custom includes. -->
-  <!-- <xacro:include filename="$(optenv JACKAL_URDF_EXTRAS empty.urdf)" /> -->
-  <!-- <xacro:include filename="$(find velodyne_description)/urdf/VLP-16.urdf.xacro"/>
-  <VLP-16 parent="rear_mount" name="velodyne" topic="/velodyne_points">
-    <origin xyz="0 0 0.4" rpy="0 0 0" />
-  </VLP-16> -->
+  <!-- Macros to generate standoffs for offset payload mounting. -->
+  <!-- <xacro:include filename="accessories/standoffs.urdf.xacro" /> -->
+  <!-- This optional plate mounts both the upgraded GPS and the Velodyne 3D LIDAR. -->
+  <xacro:include filename="accessories/bridge_plate.urdf.xacro" />
+  <!-- include camera mount for Flea3 -->
+  <xacro:include filename="accessories/camera_mount.urdf.xacro" />
+  <!-- include machine vision camera -->
+  <xacro:include filename="$(find pointgrey_camera_description)/urdf/pointgrey_flea3.urdf.xacro" />
+  <!-- Velodyne URDF, plugin, etc -->
+  <xacro:include filename="$(find velodyne_description)/urdf/VLP-16.urdf.xacro"/>
+  <VLP-16 parent="front_mount" name="velodyne" topic="/velodyne_points">
+    <origin xyz="0 0 0.05" rpy="0 0 0" />
+  </VLP-16>
 </robot>

Commit message: forgot to push all of this

File: urdf/jackal.urdf.xacro (robot description, xacro)
@@ -132,5 +132,5 @@
   </joint>
   <!-- TODO: Same note as applies to imu_link -->
-  <!-- <link name="navsat_link">
+  <link name="navsat_link">
     <visual>
       <geometry>
@@ -145,5 +145,5 @@
     <child link="navsat_link" />
     <origin xyz="-0.180 0.126 0.1815" />
-  </joint> -->
+  </joint>
   <link name="mid_mount"></link>
   <joint name="mid_mount_joint" type="fixed">

Commit message: works slightly better, no ground plane interference for the moment, pointcloud_to_laserscan working, costmap parameters tuned a bit better, but still runs into walls like it don't care

File: urdf/jackal.urdf.xacro (robot description, xacro)
@@ -6,4 +6,6 @@
   <xacro:property name="wheel_vertical_offset" value="0.0345" />
   <xacro:property name="footprint_vertical_offset" value="-0.0655" />
+  <!-- <xacro:property name="footprint_vertical_offset" value="-0.067" /> -->
+  <!-- <xacro:property name="footprint_vertical_offset" value="-0.1325" /> -->
   <xacro:property name="wheel_radius" value="0.098" />
   <xacro:property name="wheel_width" value="0.040" />
@@ -76,5 +78,6 @@
   <link name="base_link"></link>
   <joint name="base_link_joint" type="fixed">
-    <origin xyz="0 0 0" rpy="0 0 0" />
+    <!-- <origin xyz="0 0 0" rpy="0 0 0" /> -->
+    <origin xyz="0 0 0.067" rpy="0 0 0" />
     <parent link="base_link"/>
     <child link="chassis_link" />
@@ -198,5 +201,5 @@
   <xacro:include filename="$(find velodyne_description)/urdf/VLP-16.urdf.xacro"/>
   <VLP-16 parent="front_mount" name="velodyne" topic="/velodyne_points">
-    <origin xyz="0 0 0.05" rpy="0 0 0" />
+    <origin xyz="0 0 0.049" rpy="0 0 0" />
   </VLP-16>
 </robot>

Commit message: added Velodyne mount to URDF

File: urdf/jackal.urdf.xacro (robot description, xacro)
@@ -203,3 +203,20 @@
     <origin xyz="0 0 0.049" rpy="0 0 0" />
   </VLP-16>
+  <!-- Velodyne mount stuff -->
+  <link name="velodyne_mount">
+    <visual>
+      <origin xyz="0 0 -0.037" rpy="0.0 0.0 0.0" />
+      <geometry>
+        <mesh filename="package://winter_project/urdf/velodyne_mount.STL"/>
+      </geometry>
+      <material name="aluminum" >
+        <color rgba="0.45 0.45 0.45 1"/>
+      </material>
+    </visual>
+  </link>
+  <joint name="velodyne_mount_joint" type="fixed">
+    <parent link="velodyne" />
+    <child link="velodyne_mount" />
+    <origin xyz="0 0 0" />
+  </joint>
 </robot>

Commit message: renamed package to nu_jackal_autonav, updated relevant lines in all files

File: urdf/jackal.urdf.xacro (robot description, xacro)
@@ -208,5 +208,5 @@
       <origin xyz="0 0 -0.037" rpy="0.0 0.0 0.0" />
       <geometry>
-        <mesh filename="package://winter_project/urdf/velodyne_mount.STL"/>
+        <mesh filename="package://nu_jackal_autonav/urdf/velodyne_mount.STL"/>
       </geometry>
       <material name="aluminum" >

Commit message: updated velodyne mount plate relations to actually make sense

File: urdf/jackal.urdf.xacro (robot description, xacro)
@@ -206,5 +206,5 @@
   <link name="velodyne_mount">
     <visual>
-      <origin xyz="0 0 -0.037" rpy="0.0 0.0 0.0" />
+      <origin xyz="0 0 0" rpy="0.0 0.0 0.0" />
       <geometry>
         <mesh filename="package://nu_jackal_autonav/urdf/velodyne_mount.STL"/>
@@ -216,5 +216,5 @@
   </link>
   <joint name="velodyne_mount_joint" type="fixed">
-    <parent link="velodyne" />
+    <parent link="velodyne_base_link" />
     <child link="velodyne_mount" />
     <origin xyz="0 0 0" />

Commit message: more cleanup - essentially done with renaming and tidying code for now

File: urdf/jackal.urdf.xacro (robot description, xacro)
@@ -201,5 +201,5 @@
   <xacro:include filename="$(find velodyne_description)/urdf/VLP-16.urdf.xacro"/>
   <VLP-16 parent="front_mount" name="velodyne" topic="/velodyne_points">
-    <origin xyz="0 0 0.049" rpy="0 0 0" />
+    <origin xyz="0 0 0.052" rpy="0 0 0" />
   </VLP-16>
   <!-- Velodyne mount stuff -->
@@ -208,5 +208,5 @@
       <origin xyz="0 0 0" rpy="0.0 0.0 0.0" />
       <geometry>
-        <mesh filename="package://nu_jackal_autonav/urdf/velodyne_mount.STL"/>
+        <mesh filename="package://nu_jackal_autonav/urdf/velodyne_mount.stl"/>
       </geometry>
       <material name="aluminum" >
